Commit message: Updated launch file to save map in /maps directory

File: turtlebot2_description/robots/kobuki_hexagons_kinect.urdf.xacro (robot description, xacro)
@@ -1,5 +1,5 @@
 <?xml version="1.0"?>
 <robot name="turtlebot" xmlns:xacro="http://ros.org/wiki/xacro">
-  <xacro:include filename="$(find kobuki_description)/urdf/kobuki.urdf.xacro" />
+  <xacro:include filename="$(find turtlebot2_description)/urdf/kobuki/kobuki.urdf.xacro" />
   <xacro:include filename="$(find turtlebot2_description)/urdf/stacks/hexagons.urdf.xacro" />
   <xacro:include filename="$(find turtlebot2_description)/urdf/sensors/kinect.urdf.xacro"/>

File: turtlebot2_description/urdf/sensors/kinect.urdf.xacro (robot description, xacro)
@@ -3,6 +3,4 @@
   <xacro:include filename="$(find turtlebot2_description)/urdf/turtlebot_gazebo.urdf.xacro"/>
   <xacro:include filename="$(find turtlebot2_description)/urdf/turtlebot_properties.urdf.xacro"/>
-  <xacro:arg name="namespace" default=""/>
-  <xacro:property name="robot_namespace" value="/$(arg namespace)"/>
   <xacro:property name="kinect_cam_py" value="-0.0125"/>
   <!-- Parameterised in part by the values in turtlebot_properties.urdf.xacro -->

File: turtlebot2_description/urdf/turtlebot_gazebo.urdf.xacro (robot description, xacro)
@@ -7,5 +7,5 @@
     <gazebo reference="camera_link">
       <sensor type="depth" name="camera1">
-          <update_rate>20</update_rate>
+          <update_rate>30</update_rate>
           <visualize>true</visualize>
           <camera>
@@ -19,6 +19,6 @@
             </depth_camera>
             <clip>
-              <near>0.05</near>
-              <far>3</far>
+              <near>0.5</near>
+              <far>7</far>
             </clip>
             <noise>
@@ -47,4 +47,6 @@
               <remapping>mycamera/depth/image_raw/theora:=depth/image_raw/theora</remapping>
             </ros>
+            <body_name>kinect_rgb</body_name>
+            <frame_name>kinect_rgb</frame_name>
             <!-- omit camera_name to default to sensor name -->
             <camera_name>mycamera</camera_name>
@@ -54,5 +56,5 @@
           </plugin>
           <always_on>true</always_on>
-          <frame_name>camera_link</frame_name>
+          >
         </sensor>
     </gazebo>
