Commit message: fix gazebo + rtabmap

File: turtlebot2_description/urdf/kobuki/kobuki.urdf.xacro (robot description, xacro)
@@ -7,5 +7,5 @@
  -->
 <robot name="kobuki" xmlns:xacro="http://ros.org/wiki/xacro">
-  <xacro:include filename="$(find kobuki_description)/urdf/common_properties.urdf.xacro"/>
+  <xacro:include filename="$(find turtlebot2_description)/urdf/common_properties.urdf.xacro"/>
   <xacro:include filename="$(find turtlebot2_description)/urdf/kobuki/kobuki_gazebo.urdf.xacro"/>
   <!-- Kobuki -->

File: turtlebot2_description/urdf/kobuki/kobuki_gazebo.urdf.xacro (robot description, xacro)
@@ -1,7 +1,7 @@
 <?xml version="1.0"?>
 <robot name="kobuki_sim" xmlns:xacro="http://ros.org/wiki/xacro">
-  <xacro:macro name="kobuki_sim">
   <xacro:arg name="namespace" default="turtlebot"/>
   <xacro:property name="robot_namespace" value="/$(arg namespace)"/>
+  <xacro:macro name="kobuki_sim">
 	  <gazebo reference="wheel_left_link">
 	    <mu1>1.0</mu1>
@@ -142,6 +142,6 @@
         <plugin name="gazebo_ros_imu_controller" filename="libgazebo_ros_imu_sensor.so">
           <ros>
-		  	<namespace>${robot_namespace}</namespace>
-            <remapping>~/out:=imu</remapping>
+		   	<namespace>${robot_namespace}</namespace>
+			<remapping>~/out:=sensor/imu_data</remapping>
           </ros>
           <output_type>sensor_msgs/msg/Imu</output_type>
@@ -180,14 +180,13 @@
         <max_wheel_torque>1.0</max_wheel_torque>
         <max_wheel_acceleration>1.0</max_wheel_acceleration>
-        <command_topic>cmd_vel</command_topic>
+		<ros>
+		   	<namespace>${robot_namespace}</namespace>
+        </ros>
+		<command_topic>cmd_vel</command_topic>
         <!-- output -->
-		<ros>
-			<namespace>${robot_namespace}</namespace>
-			<remapping>odom:=odom_turtle</remapping>
-		</ros>
         <publish_odom>true</publish_odom>
         <publish_odom_tf>true</publish_odom_tf>
         <publish_wheel_tf>true</publish_wheel_tf>
-        <odometry_topic>odom</odometry_topic>
+        <odometry_topic>odom_turtle</odometry_topic>
         <odometry_frame>odom</odometry_frame>
         <robot_base_frame>base_link</robot_base_frame>

File: turtlebot2_description/urdf/turtlebot_gazebo.urdf.xacro (robot description, xacro)
@@ -56,5 +56,4 @@
           </plugin>
           <always_on>true</always_on>
-          >
         </sensor>
     </gazebo>
